File: pcb/_autosave-pcb.kicad_pcb (KiCad board)
At the start: 2 copper layers, 26.2 x 19 mm, 5 parts, among them J1 PINHD_1x5_Female

Commit message: worked on buttons design
Parts:
- moved J1 0.67 mm to (40.5, 55.8)
Routing:
- net Net-(LED1-VDD): track 40.0 -> 41.8 mm
- net Net-(J1-Pad5): track 2.29 -> 3.63 mm
- net Net-(LED1-DIN): track 11.1 -> 11.9 mm
Other:
- board size 26.2 x 19 mm -> 26.2 x 21.4 mm
Changed lines of the file:
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@@
-			)
-		)
-		(fp_text user "LED"
-			(at 0 -4.7 0)
-			(unlocked yes)
-			(layer "Cmts.User")
-			(effects
-				(font
-					(size 1 1)
-					(thickness 0.15)
-				)
 			)
 		)
@@
 	(footprint "PCM_4ms_Connector:Pins_1x05_2.54mm_TH"
 		(layer "B.Cu")
-		(at 40.4813 56.4614 90)
+		(at 40.4813 55.7937 90)
 		(descr "Through hole pin header")
 		(tags "pin header")
@@
 		)
 	)
+	(gr_line
+		(start 50.0063 75.009375)
+		(end 50.0063 67.865624)
+		(stroke
+			(width 0.05)
+			(type default)
+		)
+		(layer "Edge.Cuts")
+	)
 	(gr_arc
 		(start 50.00625 60.721875)
@@
 	)
 	(gr_line
-		(start 50.00625 54.76875)
-		(end 50.00625 73.81875)
+		(start 30.9563 53.578125)
+		(end 30.9563 60.697308)
 		(stroke
 			(width 0.05)
@@
 	)
 	(gr_line
-		(start 30.95625 54.76875)
-		(end 50.00625 54.76875)
-		(stroke
-			(width 0.05)
-			(type default)
-		)
-		(layer "Edge.Cuts")
-	)
-	(gr_line
-		(start 30.95625 73.81875)
-		(end 30.95625 54.76875)
+		(start 30.95625 53.578125)
+		(end 50.00625 53.578125)
 		(stroke
 			(width 0.05)
@@
 	)
 	(gr_line
-		(start 50.00625 73.81875)
-		(end 30.95625 73.81875)
+		(start 50.00625 53.578125)
+		(end 50.00625 60.721875)
 		(stroke
 			(width 0.05)
@@
 		(layer "Edge.Cuts")
 	)
+	(gr_line
+		(start 50.00625 75.009375)
+		(end 30.95625 75.009375)
+		(stroke
+			(width 0.05)
+			(type default)
+		)
+		(layer "Edge.Cuts")
+	)
+	(gr_line
+		(start 30.95625 67.890192)
+		(end 30.95625 75.009375)
+		(stroke
+			(width 0.05)
+			(type default)
+		)
+		(layer "Edge.Cuts")
+	)
 	(segment
 		(start 38.1372 71.8454)
@@
 	)
 	(segment
-		(start 44.396 66.329)
-		(end 40.4813 70.2437)
+		(start 41.671875 66.904655)
+		(end 39.06097 66.904655)
 		(width 0.2)
 		(layer "B.Cu")
@@
 	)
 	(segment
-		(start 44.396 56.4614)
-		(end 44.396 66.329)
+		(start 45.5613 56.4614)
+		(end 45.5613 63.01523)
 		(width 0.2)
 		(layer "B.Cu")
@@
 	)
 	(segment
-		(start 45.5613 56.4614)
-		(end 44.396 56.4614)
+		(start 45.5613 63.01523)
+		(end 41.671875 66.904655)
 		(width 0.2)
 		(layer "B.Cu")
@@
 	)
 	(segment
+		(start 39.06097 66.904655)
+		(end 38.1 67.865625)
+		(width 0.2)
+		(layer "B.Cu")
+		(net 1)
+	)
+	(segment
+		(start 38.1 67.865625)
+		(end 38.1 70.246875)
+		(width 0.2)
+		(layer "B.Cu")
+		(net 1)
+	)
+	(segment
 		(start 45.4813 67.2169)
 		(end 45.4813 68.0437)
@@
 	)
 	(segment
-		(start 32.6259 64.8956)
+		(start 44.1866 57.283475)
+		(end 44.1866 60.8583)
+		(width 0.2)
+		(layer "F.Cu")
+		(net 3)
+	)
+	(segment
+		(start 43.364525 56.4614)
+		(end 44.1866 57.283475)
+		(width 0.2)
+		(layer "F.Cu")
+		(net 3)
+	)
+	(segment
+		(start 32.6259 63.7939)
+		(end 32.6259 64.8956)
+		(width 0.2)
+		(layer "F.Cu")
+		(net 3)
+	)
+	(segment
+		(start 34.3868 62.033)
 		(end 32.6259 63.7939)
 		(width 0.2)
@@
 	)
 	(segment
-		(start 44.1866 56.4614)
-		(end 44.1866 60.8583)
+		(start 43.0213 56.4614)
+		(end 43.364525 56.4614)
+		(width 0.2)
+		(layer "F.Cu")
+		(net 3)
+	)
+	(segment
+		(start 43.0119 62.033)
+		(end 34.3868 62.033)
 		(width 0.2)
 		(layer "F.Cu")
@@
 	)
 	(segment
-		(start 34.3868 62.033)
-		(end 32.6259 63.7939)
-		(width 0.2)
-		(layer "F.Cu")
-		(net 3)
-	)
-	(segment
-		(start 43.0119 62.033)
-		(end 34.3868 62.033)
-		(width 0.2)
-		(layer "F.Cu")
-		(net 3)
-	)
-	(segment
-		(start 43.0213 56.4614)
-		(end 44.1866 56.4614)
-		(width 0.2)
-		(layer "F.Cu")
-		(net 3)
-	)
-	(segment
-		(start 40.4813 56.4614)
-		(end 41.6466 56.4614)
+		(start 43.2063 58.8437)
+		(end 43.2063 58.00022)
 		(width 0.2)
 		(layer "F.Cu")
@@
 	)
 	(segment
-		(start 41.6466 57.1321)
-		(end 41.6466 56.4614)
+		(start 43.2063 58.00022)
+		(end 41.66748 56.4614)
 		(width 0.2)
 		(layer "F.Cu")
@@
 	)
 	(segment
-		(start 43.2063 58.6918)
-		(end 41.6466 57.1321)
-		(width 0.2)
-		(layer "F.Cu")
-		(net 4)
-	)
-	(segment
-		(start 43.2063 58.8437)
-		(end 43.2063 58.6918)
+		(start 41.66748 56.4614)
+		(end 40.4813 56.4614)
 		(width 0.2)
 		(layer "F.Cu")
@@
 		(net 5)
 	)
-	(segment
-		(start 43.2063 60.8539)
-		(end 43.2063 60.3437)
-		(width 0.2)
-		(layer "F.Cu")
-		(net 6)
-	)
-	(segment
-		(start 42.5222 61.4306)
-		(end 42.6296 61.4306)
-		(width 0.2)
-		(layer "F.Cu")
-		(net 6)
-	)
-	(segment
-		(start 42.6296 61.4306)
-		(end 43.2063 60.8539)
-		(width 0.2)
-		(layer "F.Cu")
-		(net 6)
-	)
-	(segment
-		(start 42.6296 61.4306)
-		(end 42.5222 61.4306)
-		(width 0.2)
-		(layer "F.Cu")
-		(net 6)
-	)
 	(via
-		(at 42.6296 61.4306)
+		(at 43.2063 60.3437)
 		(size 0.6)
 		(drill 0.3)
@@
 	)
 	(segment
-		(start 38.7972 61.538)
-		(end 42.5222 61.538)
+		(start 38.692741 62.07485)
+		(end 37.9413 61.323409)
 		(width 0.2)
 		(layer "B.Cu")
@@
 	)
 	(segment
-		(start 37.9413 60.6821)
-		(end 38.7972 61.538)
+		(start 43.2063 60.3437)
+		(end 43.2063 61.5687)
 		(width 0.2)
 		(layer "B.Cu")
@@
 	)
 	(segment
-		(start 42.5222 61.4306)
-		(end 42.6296 61.4306)
+		(start 37.9413 61.323409)
+		(end 37.9413 56.4614)
 		(width 0.2)
 		(layer "B.Cu")
@@
 	)
 	(segment
-		(start 42.5222 61.538)
-		(end 42.6296 61.4306)
+		(start 42.70015 62.07485)
+		(end 38.692741 62.07485)
 		(width 0.2)
 		(layer "B.Cu")
@@
 	)
 	(segment
-		(start 37.9413 56.4614)
-		(end 37.9413 60.6821)
+		(start 43.2063 61.5687)
+		(end 42.70015 62.07485)
 		(width 0.2)
 		(layer "B.Cu")
@@
 	)
 	(segment
-		(start 42.6296 61.4306)
-		(end 42.5222 61.4306)
-		(width 0.2)
-		(layer "B.Cu")
-		(net 6)
+		(start 35.4013 57.7791)
+		(end 35.4428 57.8206)
+		(width 0.2)
+		(layer "F.Cu")
+		(net 7)
 	)
 	(segment
 		(start 35.4013 56.4614)
-		(end 35.4013 57.7791)
+		(end 35.4013 55.7937)
 		(width 0.2)
 		(layer "F.Cu")
@@
 	)
 	(segment
-		(start 35.4013 57.7791)
-		(end 35.4428 57.8206)
-		(width 0.2)
-		(layer "F.Cu")
+		(start 35.4013 55.7937)
+		(end 35.4013 57.7791)
+		(width 0.2)
+		(layer "F.Cu")
