File: pcb/_autosave-pcb.kicad_sch (KiCad schematic)
At the start: 7 parts, among them U1 Seeeduino Xiao rp2040

Commit message: worked on buttons design
Parts:
- removed CH1, CH2: choc_v1_SW_solder, PCM_marbastlib-choc:SW_choc_v1_1u, symbol PCM_marbastlib-choc:choc_v1_SW_solder
- removed S1, S2, S3, S4: choc_stab, PCM_marbastlib-xp-choc:STAB_choc_2u, symbol PCM_marbastlib-choc:choc_stab
- removed U1: Seeeduino Xiao rp2040, PCM_marbastlib-xp-promicroish:Xiao_rp2040_ACH, symbol PCM_marbastlib-promicroish:Seeeduino_Xiao_rp2040
- added CH1: choc_v1_SW_HS, PCM_marbastlib-choc:SW_choc_v1_HS_CPG135001S30_1u, symbol PCM_marbastlib-choc:choc_v1_SW_HS_CPG135001S30
- added D1: 1N4148, PCM_Diode_THT_AKL:D_DO-35_SOD27_P7.62mm_Horizontal, symbol PCM_Diode_AKL:1N4148
- added J1: PINHD_1x5_Female, PCM_4ms_Connector:Pins_1x05_2.54mm_TH, symbol PCM_SL_Pin_Headers:PINHD_1x5_Female
- added LED1: choc_SK6812MINI-E, PCM_marbastlib-choc:LED_choc_6028R, symbol PCM_marbastlib-choc:choc_SK6812MINI-E
- added R1: 500, PCM_4ms_Resistor:R_0603, symbol PCM_SL_Resistors:Resistor
Connections:
- new net: LED1.2 (DOUT), R1.1
- new net: J1.5, R1.2
- new net: D1.1 (K), J1.2
- new net: CH1.1, D1.2 (A)
- new net: CH1.2, J1.1, LED1.1 (VDD)
- new net: J1.3, LED1.4 (VSS)
- new net: J1.4, LED1.3 (DIN)
